File: Digit.kicad_sch (KiCad schematic)
At the start: 17 parts

Commit message: JLC: Fixup for JLC Production
Parts:
- DS60, DS61, DS62, DS63, DS64, DS65, DS66, DS67, DS68, DS69, DS70, DS71, DS72, DS73, DS74, DS75, DS76: LCSC C2761795 -> C2843785
Changed lines of the file:
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@@
       (effects (font (size 1.27 1.27)) (justify left top) hide)
     )
-    (property "LCSC" "C2761795" (at 132.08 39.37 0)
+    (property "LCSC" "C2843785" (at 132.08 39.37 0)
       (effects (font (size 1.27 1.27)) hide)
     )
@@
       (effects (font (size 1.27 1.27)) (justify left top) hide)
     )
-    (property "LCSC" "C2761795" (at 90.17 39.37 0)
+    (property "LCSC" "C2843785" (at 90.17 39.37 0)
       (effects (font (size 1.27 1.27)) hide)
     )
@@
       (effects (font (size 1.27 1.27)) (justify left top) hide)
     )
-    (property "LCSC" "C2761795" (at 171.45 39.37 0)
+    (property "LCSC" "C2843785" (at 171.45 39.37 0)
       (effects (font (size 1.27 1.27)) hide)
     )
@@
       (effects (font (size 1.27 1.27)) (justify left top) hide)
     )
-    (property "LCSC" "C2761795" (at 151.13 60.96 0)
+    (property "LCSC" "C2843785" (at 151.13 60.96 0)
       (effects (font (size 1.27 1.27)) hide)
     )
@@
       (effects (font (size 1.27 1.27)) (justify left top) hide)
     )
-    (property "LCSC" "C2761795" (at 233.68 39.37 0)
+    (property "LCSC" "C2843785" (at 233.68 39.37 0)
       (effects (font (size 1.27 1.27)) hide)
     )
@@
       (effects (font (size 1.27 1.27)) (justify left top) hide)
     )
-    (property "LCSC" "C2761795" (at 191.77 39.37 0)
+    (property "LCSC" "C2843785" (at 191.77 39.37 0)
       (effects (font (size 1.27 1.27)) hide)
     )
@@
       (effects (font (size 1.27 1.27)) (justify left top) hide)
     )
-    (property "LCSC" "C2761795" (at 171.45 60.96 0)
+    (property "LCSC" "C2843785" (at 171.45 60.96 0)
       (effects (font (size 1.27 1.27)) hide)
     )
@@
       (effects (font (size 1.27 1.27)) (justify left top) hide)
     )
-    (property "LCSC" "C2761795" (at 151.13 39.37 0)
+    (property "LCSC" "C2843785" (at 151.13 39.37 0)
       (effects (font (size 1.27 1.27)) hide)
     )
@@
       (effects (font (size 1.27 1.27)) (justify left top) hide)
     )
-    (property "LCSC" "C2761795" (at 212.09 39.37 0)
+    (property "LCSC" "C2843785" (at 212.09 39.37 0)
       (effects (font (size 1.27 1.27)) hide)
     )
@@
       (effects (font (size 1.27 1.27)) (justify left top) hide)
     )
-    (property "LCSC" "C2761795" (at 46.99 60.96 0)
+    (property "LCSC" "C2843785" (at 46.99 60.96 0)
       (effects (font (size 1.27 1.27)) hide)
     )
@@
       (effects (font (size 1.27 1.27)) (justify left top) hide)
     )
-    (property "LCSC" "C2761795" (at 46.99 39.37 0)
+    (property "LCSC" "C2843785" (at 46.99 39.37 0)
       (effects (font (size 1.27 1.27)) hide)
     )
@@
       (effects (font (size 1.27 1.27)) (justify left top) hide)
     )
-    (property "LCSC" "C2761795" (at 90.17 60.96 0)
+    (property "LCSC" "C2843785" (at 90.17 60.96 0)
       (effects (font (size 1.27 1.27)) hide)
     )
@@
       (effects (font (size 1.27 1.27)) (justify left top) hide)
     )
-    (property "LCSC" "C2761795" (at 68.58 60.96 0)
+    (property "LCSC" "C2843785" (at 68.58 60.96 0)
       (effects (font (size 1.27 1.27)) hide)
     )
@@
       (effects (font (size 1.27 1.27)) (justify left top) hide)
     )
-    (property "LCSC" "C2761795" (at 111.76 60.96 0)
+    (property "LCSC" "C2843785" (at 111.76 60.96 0)
       (effects (font (size 1.27 1.27)) hide)
     )
@@
       (effects (font (size 1.27 1.27)) (justify left top) hide)
     )
-    (property "LCSC" "C2761795" (at 111.76 39.37 0)
+    (property "LCSC" "C2843785" (at 111.76 39.37 0)
       (effects (font (size 1.27 1.27)) hide)
     )
@@
       (effects (font (size 1.27 1.27)) (justify left top) hide)
     )
-    (property "LCSC" "C2761795" (at 132.08 60.96 0)
+    (property "LCSC" "C2843785" (at 132.08 60.96 0)
       (effects (font (size 1.27 1.27)) hide)
     )
@@
       (effects (font (size 1.27 1.27)) (justify left top) hide)
     )
-    (property "LCSC" "C2761795" (at 68.58 39.37 0)
-      (effects (font (size 1.27 1.27)) hide)
-    )
+    (property "LCSC" "C2843785" (at 68.58 39.37 0)
+      (effects (font (size 1.27 1.27)) hide)
+    )
