File: LEDCircle.kicad_sch (KiCad schematic)
At the start: 60 parts

Commit message: JLC: Fixup for JLC Production
Parts:
- DS0, DS1, DS10, DS11, DS12, DS13, DS14, DS15, DS16, DS17, DS18, DS19, DS2, DS20, DS21, DS22, DS23, DS24, DS25, DS26, DS27, DS28, DS29, DS3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: LCSC C2761795 -> C2843785
- DS51: value S2812B -> WS2812B; LCSC C2761795 -> C2843785
